File: hardware/eagle/type2interface/SimulatorT2InterfaceRevC.brd (EAGLE design)
At the start: 80 x 80 mm, 25 parts, among them IC1 7805T, IC2 MAX233, IC3 ATMEGA328P_PDIP

Commit message: Minor fix to Interface board
Routing:
- net VCC: track 261.2 -> 262.4 mm
Changed lines of the file:
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@@
 <via x="24.13" y="55.88" extent="1-16" drill="0.6" diameter="0.254"/>
 <via x="39.37" y="68.58" extent="1-16" drill="0.6" diameter="0.254"/>
+<via x="24.13" y="71.12" extent="1-16" drill="0.6" diameter="0.254"/>
+<via x="20.32" y="78.74" extent="1-16" drill="0.6" diameter="0.254"/>
+<via x="20.32" y="74.93" extent="1-16" drill="0.6" diameter="0.254"/>
+<via x="20.32" y="71.12" extent="1-16" drill="0.6" diameter="0.254"/>
 </signal>
 <signal name="VCC">
@@
 <wire x1="25.4" y1="53.34" x2="35.56" y2="43.18" width="0.6096" layer="16"/>
 <wire x1="35.56" y1="43.18" x2="35.56" y2="40.64" width="0.6096" layer="16"/>
-<wire x1="24.0792" y1="53.3908" x2="22.86" y2="53.4416" width="0.6096" layer="16"/>
-<wire x1="22.86" y1="53.4416" x2="22.86" y2="63.0555" width="0.6096" layer="16"/>
-<wire x1="22.86" y1="63.0555" x2="24.13" y2="63.0428" width="0.6096" layer="16"/>
+<wire x1="24.0792" y1="53.3908" x2="21.59" y2="53.4416" width="0.6096" layer="16"/>
+<wire x1="21.59" y1="53.4416" x2="21.59" y2="63.0555" width="0.6096" layer="16"/>
+<wire x1="21.59" y1="63.0555" x2="24.13" y2="63.0428" width="0.6096" layer="16"/>
 <wire x1="73.66" y1="63.119" x2="73.66" y2="61.087" width="0.6096" layer="16"/>
 <wire x1="73.66" y1="61.087" x2="76.2" y2="61.087" width="0.6096" layer="16"/>
@@
 <wire x1="73.66" y1="29.591" x2="76.2" y2="29.591" width="0.6096" layer="16"/>
 <wire x1="73.66" y1="45.339" x2="76.2" y2="45.339" width="0.6096" layer="16"/>
-<wire x1="16.764" y1="63.0555" x2="22.86" y2="63.0555" width="0.1524" layer="16"/>
+<wire x1="16.764" y1="63.0555" x2="21.59" y2="63.0555" width="0.1524" layer="16"/>
 </signal>
 <signal name="MOSI">
