File: hardware/eagle/type2interface/SimulatorT2InterfaceRevE.sch (EAGLE design)
At the start: 25 parts, among them IC1 7805T, IC2 MAX233, IC3 ATMEGA328P_PDIP

Commit message: Interface RevE Boards
Eagle files and Gerbers for Type 2 Interface Board Rev E
Parts:
- added Q1: CSTLS8M00G53-B0, murata-resonators:CSTLS_G
Connections:
- new net OSC1: IC3.PB6(XTAL1/TOSC1), Q1.1
- new net OSC2: IC3.PB7(XTAL2/TOSC2), Q1.3
- net GND: now also Q1.GND
Changed lines of the file:
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@@
 <part name="FRAME1" library="SparkFun-Aesthetics" deviceset="FRAME-A4L" device="">
 <attribute name="CNAME" value="Liverpool Simulator Type 2 Interface"/>
-<attribute name="CREVISION" value="Rev D 01/2019"/>
+<attribute name="CREVISION" value="Rev E 05/2019"/>
 <attribute name="DESIGNER" value="A J Instone-Cowie"/>
 </part>
@@
 <part name="PC" library="AIC_Custom" deviceset="RJ45-RJHSE-5084" device=""/>
 <part name="TP7" library="SparkFun-Connectors" deviceset="M01" device="PTH"/>
+<part name="Q1" library="murata-resonators" deviceset="CSTLS_G" device="" value="CSTLS8M00G53-B0"/>
 </parts>
 <sheets>
@@
 <instance part="PC" gate="G$1" x="22.86" y="121.92" rot="MR0"/>
 <instance part="TP7" gate="G$1" x="177.8" y="33.02"/>
+<instance part="Q1" gate="G$1" x="127" y="106.68"/>
 </instances>
 <busses>
@@
 <wire x1="142.24" y1="81.28" x2="137.16" y2="81.28" width="0.1524" layer="91"/>
 <junction x="137.16" y="81.28"/>
+<pinref part="Q1" gate="G$1" pin="GND"/>
+<wire x1="127" y1="99.06" x2="127" y2="81.28" width="0.1524" layer="91"/>
+<wire x1="127" y1="81.28" x2="137.16" y2="81.28" width="0.1524" layer="91"/>
 </segment>
 <segment>
@@
 </segment>
 </net>
+<net name="OSC2" class="0">
+<segment>
+<pinref part="Q1" gate="G$1" pin="3"/>
+<pinref part="IC3" gate="G$1" pin="PB7(XTAL2/TOSC2)"/>
+<wire x1="132.08" y1="106.68" x2="142.24" y2="106.68" width="0.1524" layer="91"/>
+</segment>
+</net>
+<net name="OSC1" class="0">
+<segment>
+<pinref part="IC3" gate="G$1" pin="PB6(XTAL1/TOSC1)"/>
+<wire x1="142.24" y1="111.76" x2="119.38" y2="111.76" width="0.1524" layer="91"/>
+<wire x1="119.38" y1="111.76" x2="119.38" y2="106.68" width="0.1524" layer="91"/>
+<pinref part="Q1" gate="G$1" pin="1"/>
+<wire x1="119.38" y1="106.68" x2="121.92" y2="106.68" width="0.1524" layer="91"/>
+</segment>
+</net>
