File: hardware/eagle/type2power/SimulatorT2PowerRevC.sch (EAGLE design)
At the start: 7 parts

Commit message: Power Board Rev C
Add an indication of power supply polarity to the top silkscreen.
Connections:
- net P6 renamed TX2
Changed lines of the file:
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@@
 <part name="FRAME1" library="SparkFun-Aesthetics" deviceset="FRAME-A4L" device="">
 <attribute name="CNAME" value="Simulator Type 2 Power"/>
-<attribute name="CREVISION" value="Rev B 03/2018"/>
+<attribute name="CREVISION" value="Rev C 02/2019"/>
 <attribute name="DESIGNER" value="A J Instone-Cowie"/>
 </part>
@@
 </segment>
 </net>
-<net name="P6" class="0">
+<net name="TX2" class="0">
 <segment>
 <pinref part="TP1" gate="G$1" pin="3"/>
