File: hardware/eagle/type2secondpc/SimulatorT2SecondPCRevA_panel4.brd (EAGLE design)
At the start: 99.1 x 99.1 mm, 28 parts

Commit message: Board fixes
Parts:
- moved E$8 71.1 mm to (49.5, 85.1)
- moved E$6 50.8 mm to (49.5, 14.0)
- moved E$5 49.5 mm to (49.5, 34.3)
- moved E$7 30.5 mm to (49.5, 64.8)
Other:
- outline, holes or cut-outs redrawn
- board text added: "POWER BOARD INTERFACE"
- board text removed: "Power Board Interface"
Changed lines of the file:
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@@
 <layer number="23" name="tOrigins" color="15" fill="1" visible="yes" active="yes"/>
 <layer number="24" name="bOrigins" color="15" fill="1" visible="yes" active="yes"/>
-<layer number="25" name="tNames" color="7" fill="1" visible="no" active="yes"/>
+<layer number="25" name="tNames" color="7" fill="1" visible="yes" active="yes"/>
 <layer number="26" name="bNames" color="7" fill="1" visible="yes" active="yes"/>
-<layer number="27" name="tValues" color="7" fill="1" visible="yes" active="yes"/>
-<layer number="28" name="bValues" color="7" fill="1" visible="yes" active="yes"/>
+<layer number="27" name="tValues" color="7" fill="1" visible="no" active="yes"/>
+<layer number="28" name="bValues" color="7" fill="1" visible="no" active="yes"/>
 <layer number="29" name="tStop" color="7" fill="3" visible="no" active="yes"/>
 <layer number="30" name="bStop" color="7" fill="6" visible="no" active="yes"/>
@@
 <layer number="124" name="bTestmark" color="7" fill="1" visible="no" active="yes"/>
 <layer number="125" name="_tNames" color="14" fill="1" visible="yes" active="yes"/>
-<layer number="126" name="_bNames" color="7" fill="1" visible="no" active="yes"/>
+<layer number="126" name="_bNames" color="7" fill="1" visible="yes" active="yes"/>
 <layer number="127" name="_tValues" color="7" fill="1" visible="no" active="yes"/>
 <layer number="128" name="_bValues" color="7" fill="1" visible="no" active="yes"/>
@@
 <wire x1="45.72" y1="0" x2="2.54" y2="0" width="0.4064" layer="20"/>
 <wire x1="2.54" y1="0" x2="0" y2="2.54" width="0.4064" layer="20" curve="-90"/>
-<text x="33.02" y="23.495" size="1.27" layer="21" font="vector" rot="R90" align="bottom-center">Power Board    Interface</text>
+<text x="33.02" y="23.495" size="1.27" layer="21" font="vector" rot="R90" align="bottom-center">POWER BOARD    INTERFACE</text>
 <text x="17.78" y="24.13" size="1.27" layer="21" font="vector" rot="R90" align="bottom-center">REQUIRES INTERFACE BOARD
 REV D OR LATER</text>
@@
 <text x="76.835" y="3.81" size="1.27" layer="21" font="vector" align="center">Rev A
 04/2019</text>
-<dimension x1="100.33" y1="99.06" x2="100.33" y2="0" x3="106.68000625" y3="49.53" textsize="1.778" layer="47"/>
 <wire x1="50.8" y1="45.72" x2="53.34" y2="48.26" width="0.4064" layer="20" curve="-90"/>
 <wire x1="96.52" y1="48.26" x2="99.06" y2="45.72" width="0.4064" layer="20" curve="-90"/>
@@
 <wire x1="96.52" y1="0" x2="53.34" y2="0" width="0.4064" layer="20"/>
 <wire x1="53.34" y1="0" x2="50.8" y2="2.54" width="0.4064" layer="20" curve="-90"/>
-<text x="83.82" y="23.495" size="1.27" layer="21" font="vector" rot="R90" align="bottom-center">Power Board    Interface</text>
+<text x="83.82" y="23.495" size="1.27" layer="21" font="vector" rot="R90" align="bottom-center">POWER BOARD    INTERFACE</text>
 <text x="68.58" y="24.13" size="1.27" layer="21" font="vector" rot="R90" align="bottom-center">REQUIRES INTERFACE BOARD
 REV D OR LATER</text>
@@
 <wire x1="48.26" y1="53.34" x2="45.72" y2="50.8" width="0.4064" layer="20" curve="-90"/>
 <wire x1="2.54" y1="50.8" x2="0" y2="53.34" width="0.4064" layer="20" curve="-90"/>
-<text x="33.02" y="74.295" size="1.27" layer="21" font="vector" rot="R90" align="bottom-center">Power Board    Interface</text>
+<text x="33.02" y="74.295" size="1.27" layer="21" font="vector" rot="R90" align="bottom-center">POWER BOARD    INTERFACE</text>
 <text x="17.78" y="74.93" size="1.27" layer="21" font="vector" rot="R90" align="bottom-center">REQUIRES INTERFACE BOARD
 REV D OR LATER</text>
@@
 <text x="76.835" y="54.61" size="1.27" layer="21" font="vector" align="center">Rev A
 04/2019</text>
+<dimension x1="100.33" y1="99.06" x2="100.33" y2="0" x3="106.68000625" y3="49.53" textsize="1.778" layer="47"/>
 <wire x1="50.8" y1="96.52" x2="53.34" y2="99.06" width="0.4064" layer="20" curve="-90"/>
 <wire x1="53.34" y1="99.06" x2="96.52" y2="99.06" width="0.4064" layer="20"/>
@@
 <wire x1="99.06" y1="53.34" x2="96.52" y2="50.8" width="0.4064" layer="20" curve="-90"/>
 <wire x1="53.34" y1="50.8" x2="50.8" y2="53.34" width="0.4064" layer="20" curve="-90"/>
-<text x="83.82" y="74.295" size="1.27" layer="21" font="vector" rot="R90" align="bottom-center">Power Board    Interface</text>
+<text x="83.82" y="74.295" size="1.27" layer="21" font="vector" rot="R90" align="bottom-center">POWER BOARD    INTERFACE</text>
 <text x="68.58" y="74.93" size="1.27" layer="21" font="vector" rot="R90" align="bottom-center">REQUIRES INTERFACE BOARD
 REV D OR LATER</text>
@@
 <wire x1="83.82" y1="48.26" x2="66.04" y2="48.26" width="0.4064" layer="20"/>
 <wire x1="66.04" y1="48.26" x2="66.04" y2="50.8" width="0.4064" layer="20"/>
-<wire x1="48.26" y1="96.52" x2="48.26" y2="85.09" width="0.4064" layer="20"/>
-<wire x1="48.26" y1="85.09" x2="50.8" y2="85.09" width="0.4064" layer="20"/>
-<wire x1="50.8" y1="85.09" x2="50.8" y2="96.52" width="0.4064" layer="20"/>
+<wire x1="48.26" y1="96.52" x2="48.26" y2="86.36" width="0.4064" layer="20"/>
+<wire x1="48.26" y1="86.36" x2="50.8" y2="86.36" width="0.4064" layer="20"/>
+<wire x1="50.8" y1="86.36" x2="50.8" y2="96.52" width="0.4064" layer="20"/>
 <wire x1="48.26" y1="53.34" x2="48.26" y2="63.5" width="0.4064" layer="20"/>
 <wire x1="48.26" y1="63.5" x2="50.8" y2="63.5" width="0.4064" layer="20"/>
 <wire x1="50.8" y1="63.5" x2="50.8" y2="53.34" width="0.4064" layer="20"/>
-<wire x1="48.26" y1="82.55" x2="50.8" y2="82.55" width="0.4064" layer="20"/>
-<wire x1="50.8" y1="82.55" x2="50.8" y2="66.04" width="0.4064" layer="20"/>
+<wire x1="48.26" y1="83.82" x2="50.8" y2="83.82" width="0.4064" layer="20"/>
+<wire x1="50.8" y1="83.82" x2="50.8" y2="66.04" width="0.4064" layer="20"/>
 <wire x1="50.8" y1="66.04" x2="48.26" y2="66.04" width="0.4064" layer="20"/>
-<wire x1="48.26" y1="66.04" x2="48.26" y2="82.55" width="0.4064" layer="20"/>
+<wire x1="48.26" y1="66.04" x2="48.26" y2="83.82" width="0.4064" layer="20"/>
 <wire x1="48.26" y1="45.72" x2="48.26" y2="35.56" width="0.4064" layer="20"/>
 <wire x1="48.26" y1="35.56" x2="50.8" y2="35.56" width="0.4064" layer="20"/>
@@
 <wire x1="48.26" y1="12.7" x2="50.8" y2="12.7" width="0.4064" layer="20"/>
 <wire x1="50.8" y1="12.7" x2="50.8" y2="2.54" width="0.4064" layer="20"/>
-<wire x1="48.26" y1="33.02" x2="50.8" y2="33.02" width="0.4064" layer="20"/>
 <wire x1="50.8" y1="33.02" x2="50.8" y2="15.24" width="0.4064" layer="20"/>
 <wire x1="50.8" y1="15.24" x2="48.26" y2="15.24" width="0.4064" layer="20"/>
 <wire x1="48.26" y1="15.24" x2="48.26" y2="33.02" width="0.4064" layer="20"/>
-<text x="74.93" y="49.53" size="1.016" layer="20" align="center">CUT OUT</text>
-<text x="49.53" y="49.53" size="1.016" layer="20" align="center">CUT OUT</text>
-<text x="24.13" y="49.53" size="1.016" layer="20" align="center">CUT OUT</text>
-<text x="49.53" y="74.93" size="1.016" layer="20" rot="R90" align="center">CUT OUT</text>
-<text x="49.53" y="24.13" size="1.016" layer="20" rot="R90" align="center">CUT OUT</text>
+<wire x1="48.26" y1="33.02" x2="50.8" y2="33.02" width="0.4064" layer="20"/>
+<text x="49.53" y="49.53" size="1.016" layer="20" font="vector" align="center">CUT OUT</text>
+<text x="74.93" y="49.53" size="1.016" layer="20" font="vector" align="center">CUT OUT</text>
+<text x="24.13" y="49.53" size="1.016" layer="20" font="vector" align="center">CUT OUT</text>
+<text x="49.53" y="24.13" size="1.016" layer="20" font="vector" rot="R270" align="center">CUT OUT</text>
+<text x="49.53" y="74.93" size="1.016" layer="20" font="vector" rot="R90" align="center">CUT OUT</text>
 </plain>
 <attributes>
@@
 <element name="E$3" library="AIC_Custom" package="STAMP_HOLES" value="" x="64.77" y="49.53"/>
 <element name="E$4" library="AIC_Custom" package="STAMP_HOLES" value="" x="85.09" y="49.53"/>
-<element name="E$5" library="AIC_Custom" package="STAMP_HOLES" value="" x="49.53" y="83.82" rot="R90"/>
-<element name="E$6" library="AIC_Custom" package="STAMP_HOLES" value="" x="49.53" y="64.77" rot="R90"/>
-<element name="E$7" library="AIC_Custom" package="STAMP_HOLES" value="" x="49.53" y="34.29" rot="R90"/>
-<element name="E$8" library="AIC_Custom" package="STAMP_HOLES" value="" x="49.53" y="13.97" rot="R90"/>
+<element name="E$5" library="AIC_Custom" package="STAMP_HOLES" value="" x="49.53" y="34.29" rot="R90"/>
+<element name="E$6" library="AIC_Custom" package="STAMP_HOLES" value="" x="49.53" y="13.97" rot="R90"/>
+<element name="E$7" library="AIC_Custom" package="STAMP_HOLES" value="" x="49.53" y="64.77" rot="R90"/>
+<element name="E$8" library="AIC_Custom" package="STAMP_HOLES" value="" x="49.53" y="85.09" rot="R90"/>
 </elements>
 <signals>
